File: sensor_card/sensor_card.kicad_sch (KiCad schematic)
At the start: 18 parts, among them J1 Raspberry_Pi_4, J10 Conn_01x05, J2 BME280, J3 GPS, J4 PARACHUTE, J5 Conn_01x02, J6 power LORA, J7 power_RPI, J8 MPU_6500, U1 Ai-Thinker-Ra-02

Commit message: sensor card: full revision
Parts:
- removed H1, H6, H7, H8: MountingHole_RPI, MountingHole:MountingHole_2.2mm_M2_DIN965_Pad, symbol Mechanical:MountingHole_Pad
- removed H2, H3, H4, H5: MountingHole_Pad, MountingHole:MountingHole_3.2mm_M3_DIN965_Pad, symbol Mechanical:MountingHole_Pad
- removed J2: BME280, PHOENIX:BME 280, symbol Connector_Generic:Conn_01x04
- added J12: AIRBRAKE, Connector_JST:JST_XH_S4B-XH-A_1x04_P2.50mm_Horizontal, symbol Connector_Generic:Conn_01x04
- added J2: BME, nasa:BME280, symbol Connector_Generic:Conn_01x06
- added J8: lauch, Connector_JST:JST_XH_S2B-XH-A_1x02_P2.50mm_Horizontal, symbol Connector_Generic:Conn_01x02
- added J9: proto_selector, Connector_PinHeader_2.54mm:PinHeader_2x02_P2.54mm_Vertical, symbol Connector_Generic:Conn_02x02_Odd_Even
- added R1: 10k, Resistor_THT:R_Axial_DIN0204_L3.6mm_D1.6mm_P7.62mm_Horizontal, symbol Device:R
- J1: renamed from J5; value Conn_01x02 -> fan_power; footprint Connector_JST:JST_XH_S2B-XH-A_1x02_P2.50mm_Horizontal -> Connector_PinHeader_2.54mm:PinHeader_1x02_P2.54mm_Horizontal
- J10: renamed from J7; footprint Connector_JST:JST_XH_S4B-XH-A-1_1x04_P2.50mm_Horizontal -> Connector_JST:JST_XH_S4B-XH-A_1x04_P2.50mm_Horizontal
- J11: renamed from J6; footprint Connector_JST:JST_XH_S4B-XH-A-1_1x04_P2.50mm_Horizontal -> Connector_JST:JST_XH_S4B-XH-A_1x04_P2.50mm_Horizontal
- J3: footprint PHOENIX:GPS-MV2 -> nasa:GPS
- J6: renamed from J8; footprint PHOENIX:MPU-9250 -> nasa:MPU6500
- J7: renamed from J10; value Conn_01x05 -> hmi; footprint Connector_JST:JST_XH_S5B-XH-A-1_1x05_P2.50mm_Horizontal -> Connector_JST:JST_XH_S5B-XH-A_1x05_P2.50mm_Horizontal
- renumbered J1 to J4, J4 to J5
Connections:
- net LED_INIT_AEROFR is gone; now on net LED_PROG_WORKING: J4.26 (~{CE1}_SPI0/GPIO07)
- net +3V3: now also J3.4 (Pin_4), J7.4 (Pin_4), J2.1 (Pin_1), R1.2; no longer J3.1 (Pin_1)
- net +3V3_LORA: now also J7.2 (Pin_2)
- net +5V: now also J1.2 (Pin_2), J12.2 (Pin_2); no longer J1.1 (Pin_1)
- net GND: now also J1.1 (Pin_1), J3.1 (Pin_1), J12.1 (Pin_1), J2.2 (Pin_2), J8.1 (Pin_1); no longer J1.2 (Pin_2), J3.4 (Pin_4)
- net GPS_RX: now also J3.3 (Pin_3); no longer J3.2 (Pin_2)
- net GPS_TX: now also J3.2 (Pin_2); no longer J3.3 (Pin_3)
- net LORA_RST: now also J4.37 (GPIO26/SDIO_DAT2); no longer J4.11 (GPIO17/SPI1_~{CE1})
- net SCL: now also J2.3 (Pin_3)
- net SDA: now also J2.4 (Pin_4)
- net lauch_detect: now reaches J4.36 (GPIO16/SPI1_~{CE2})
- net lauch_detect: now also J8.2 (Pin_2), R1.1
- net LED_ALIM_AEROFR renamed LED_LORA_WORKING
- net LED_LORA_WORKING: now also J7.3 (Pin_3)
- net LED_ALIM_LORA renamed AIRBRAKE_TX_SDA
- net AIRBRAKE_TX_SDA: now also J9.4 (Pin_4); no longer J7.3 (Pin_3)
- net LED_ALIM_RPI_CAPTEURS: no longer names the net of J4.22 (GPIO25/SDIO_DAT1)
- net LED_ALIM_RPI_CAPTEURS: no longer J7.2 (Pin_2)
- net LED_FONC_LORA renamed AIRBRAKE_RX_SCL
- net AIRBRAKE_RX_SCL: now also J9.1 (Pin_1); no longer J7.4 (Pin_4)
- net LED_FONC_PROGRAMMES renamed LED_PROG_WORKING
- net LED_PROG_WORKING: no longer J4.37 (GPIO26/SDIO_DAT2)
- net PARA_STATE_FEEDBACK: no longer names the net of J4.29 (GPCLK1/GPIO05)
- net PARA_STATE_FEEDBACK: no longer J5.3 (Pin_3)
- new net: J12.3 (Pin_3), J9.2 (Pin_2)
- new net: J12.4 (Pin_4), J9.3 (Pin_3)
- new net PARACHUTE_FEEDBACK: J4.11 (GPIO17/SPI1_~{CE1}), J5.3 (Pin_3)
- no-connect marks 17 -> 20
Other:
- moved on the sheet: J7
