File: rocket/rocket.kicad_sch (KiCad schematic)
At the start: 14 parts, among them J1 Conn_01x01, J10 Conn_01x01, J11 Conn_01x01, J12 Conn_01x01, J13 Conn_01x01, J14 Conn_01x01, J2 Conn_01x01, J3 Conn_01x01, J4 Conn_01x01, J5 Conn_01x01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

Commit message: ajout d'une carte hmi
Parts:
- added J15, J16, J17, J18: Conn_01x01, symbol Connector_Generic:Conn_01x01
Connections:
- new net: J15.1 (Pin_1), J16.1 (Pin_1)
Other:
- note removed: "le signal des leds transmet la puissance"
