File: lauch_trigger/lauch_trigger.kicad_sch (KiCad schematic)
At the start: 4 parts, among them J1 jack_A, J2 conn_A, J3 jack_B, J4 conn_B

Commit message: created the pcb
Parts:
- J1: footprint (none) -> Connector_Audio:Jack_3.5mm_PJ320D_Horizontal
- J2: renamed from J3; footprint (none) -> Connector_Audio:Jack_3.5mm_PJ320D_Horizontal
- J3: renamed from J2; footprint (none) -> Connector_JST:JST_XH_B2B-XH-A_1x02_P2.50mm_Vertical
- J4: footprint (none) -> Connector_JST:JST_XH_B2B-XH-A_1x02_P2.50mm_Vertical
Other:
- moved on the sheet: J1, J2, J3, J4

Commit message: Created PCB for jack connectors
Parts:
- J1, J2: footprint Connector_Audio:Jack_3.5mm_PJ320D_Horizontal -> nasa:Jack_3.5mm_PJ320D_Horizontal
Changed lines of the file:
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@@
 			)
 		)
-		(property "Footprint" "Connector_Audio:Jack_3.5mm_PJ320D_Horizontal"
+		(property "Footprint" "nasa:Jack_3.5mm_PJ320D_Horizontal"
 			(at 106.68 95.25 0)
 			(effects
@@
 			)
 		)
-		(property "Footprint" "Connector_Audio:Jack_3.5mm_PJ320D_Horizontal"
+		(property "Footprint" "nasa:Jack_3.5mm_PJ320D_Horizontal"
 			(at 106.68 72.39 0)
 			(effects
